File: kicad/shield-periph.kicad_pcb (KiCad board)
At the start: 4 copper layers, 6 parts, among them J4 Fix, J5 Fix, J6 Fix, J7 Fix, U2 Shield_droite, U3 Shield_gauche

Commit message: Création empreinte connecteur unique et mise à jour
Parts:
- removed U2: Shield_droite, conn_shield:conn_shield
- removed U3: Shield_gauche, conn_shield:conn_shield
- added U1: Conn_shield, conn_shield:conn_shield, B.Cu at (47.0, 78.7)

Commit message: Mise en conformité avec la carte periph
Parts:
- removed J4, J5, J6, J7: Fix, Mounting_Holes:MountingHole_3.2mm_M3_Pad
- U1: moved to F.Cu
- moved U1 3.09 mm to (46.5, 81.8), turned to 0 degrees
Routing:
- removed copper zone on In2.Cu, net +3V3
- removed copper zone on B.Cu, net GND
